File: WattMeter.sch (KiCad schematic (older format))
At the start: 0 parts

Commit message: Added ACS711
Parts:
- added U?: ACS711, symbol ACS711
Changed lines of the file:
@@
 EESchema Schematic File Version 2
+LIBS:MyComponents
 LIBS:power
 LIBS:device
@@
 LIBS:contrib
 LIBS:valves
+LIBS:WattMeter-cache
 EELAYER 25 0
 EELAYER END
@@
 Comment4 ""
 $EndDescr
+$Comp
+L ACS711 U?
+U 1 1 5511C6C0
+P 3650 2650
+F 0 "U?" H 3450 2350 60  0000 C CNN
+F 1 "ACS711" H 3600 2900 60  0000 C CNN
+F 2 "" H 3650 2650 60  0000 C CNN
+F 3 "" H 3650 2650 60  0000 C CNN
+	1    3650 2650
+	1    0    0    -1
+$EndComp
 $EndSCHEMATC
